File: enzo.kicad_sch (KiCad schematic)
At the start: 61 parts, among them J3 BATTERY_CONN_DEANS, J5 S3B-PH-SM4-TB(LF)(SN), SW1 SW_Push, SW10 SW_Push, SW11 SW_Push, SW12 SW_Push, SW13 SW_Push, SW14 SW_Push, SW15 SW_Push, SW16 SW_Push, SW17 SW_Push, SW2 SW_Push, SW26 SW_SPST, SW3 SW_Push, SW4 SW_Push, SW5 SW_Push, SW6 SW_Push, SW7 SW_Push, SW8 SW_Push, SW9 SW_Push

Commit message: Fix schematics
Parts:
- removed J5: S3B-PH-SM4-TB(LF)(SN), local-libraries:JST_SH_BM02B-SRSS-TB_1x02-1MP_P1.00mm_Vertical, symbol Connector:Conn_01x02_Female
- removed JP_batt_F, JP_grnd_B: Jumper_2_Open, local-libraries:SolderJumper-2_P1.3mm_Open_RoundedPad1.0x1.5mm, symbol Jumper:Jumper_2_Open
Connections:
- net GND: no longer SW26.2 (B)
- net col4_mcu: now also JP_row4_B.2 (B)
- net row4_mcu: now also JP_col4_B.2 (B)
- net gnd renamed grnd
- net grnd: now also SW26.2 (B)
- no-connect marks 9 -> 17
Other:
- note removed: "3pin battery connector"
- note removed: "Battery jumpers"
- moved on the sheet: J3

Commit message: Another take at the jumper design, starting from the schematics
Parts:
- added JP_col1_B1, JP_col1_F1, JP_col2_B1, JP_col2_F1, JP_col3_B1, JP_col3_F1, JP_col4_B1, JP_col4_F1, JP_col5_B1, JP_col5_F1, JP_row1_B1, JP_row1_F1: Jumper_2_Open, local-libraries:SolderJumper-2_P1.3mm_Open_RoundedPad1.0x1.5mm, symbol Jumper:Jumper_2_Open
- gave numbers to parts that had none: 1
- renumbered JP_col1_B to JP_col1_B1, JP_col1_F to JP_col1_F1, JP_col2_B to JP_col2_B1, JP_col2_F to JP_col2_F1, JP_col3_B to JP_col3_B1, JP_col3_F to JP_col3_F1, JP_col4_B to JP_col4_B1, JP_col4_F to JP_col4_F1, JP_col5_B to JP_col5_B1, JP_col5_F to JP_col5_F1, JP_row1_B to JP_row1_B1, JP_row1_F to JP_row1_F1, JP_row2_B to JP_row2_B1, JP_row2_F to JP_row2_F1, JP_row3_B to JP_row3_B1, JP_row3_F to JP_row3_F1, JP_row4_B to JP_row4_B1, JP_row4_F to JP_row4_F1, JP_row5_B to JP_row5_B1, JP_row5_F to JP_row5_F1
Connections:
- net col1_matrix: now also JP_col1_B1.1 (A), JP_col1_F1.2 (B)
- net col1_mcu: now also JP_col1_F1.1 (A), JP_row1_F1.1 (A)
- net col2_matrix: now also JP_col2_B1.1 (A), JP_col2_F1.2 (B)
- net col2_mcu: now also JP_col2_F1.1 (A)
- net col3_matrix: now also JP_col3_B1.1 (A), JP_col3_F1.2 (B)
- net col3_mcu: now also JP_col3_F1.1 (A)
- net col4_matrix: now also JP_col4_B1.1 (A), JP_col4_F1.2 (B)
- net col4_mcu: now also JP_col4_F1.1 (A)
- net col5_matrix: now also JP_col5_B1.1 (A), JP_col5_F1.2 (B)
- net col5_mcu: now also JP_col5_F1.1 (A)
- net row1_mcu: now also JP_col1_B1.2 (B), JP_row1_B1.2 (B)
- net row2_mcu: now also JP_col2_B1.2 (B)
- net row3_mcu: now also JP_col3_B1.2 (B)
- net row4_mcu: now also JP_col4_B1.2 (B)
- new net row5_mcu_unused: JP_col5_B1.2 (B)

Commit message: Finish jumpers schematics
Parts:
- removed JP_col1_B1, JP_col1_F1, JP_col2_B1, JP_col2_F1, JP_col3_B1, JP_col3_F1, JP_col4_B1, JP_col4_F1, JP_col5_B1, JP_col5_F1, JP_row1_B1, JP_row1_F1: Jumper_2_Open, local-libraries:SolderJumper-2_P1.3mm_Open_RoundedPad1.0x1.5mm, symbol Jumper:Jumper_2_Open
- renumbered JP_row1_F1 to JP_row1_B1, JP_row1_B1 to JP_row1_F1
Connections:
- net grnd is gone; now on net GND: J3.-, SW26.2 (B)
- net col2_mcu: now also JP_row2_B1.1 (A); no longer JP_row2_B1.2 (B)
- net col3_mcu: now also JP_row3_B1.1 (A); no longer JP_row3_B1.2 (B)
- net col4_mcu: now also JP_row4_B1.1 (A); no longer JP_row4_B1.2 (B)
- net col5_mcu: now also JP_row5_B1.1 (A); no longer JP_row5_B1.2 (B)
- net row1_matrix: now also JP_row1_B1.2 (B), JP_row1_F1.1 (A)
- net row2_matrix: now also JP_row2_B1.2 (B); no longer JP_row2_B1.1 (A)
- net row3_matrix: now also JP_row3_B1.2 (B); no longer JP_row3_B1.1 (A)
- net row4_matrix: now also JP_row4_B1.2 (B); no longer JP_row4_B1.1 (A)
- net row5_mcu_unused: now also JP_row5_F1.2 (B)
- net at JP_row5_F1.1 (A): now also JP_row5_B1.2 (B); no longer JP_row5_B1.1 (A)
- no-connect marks 17 -> 14
Other:
- note added: "Matrix/MCU jumpers"
- note removed: "Column jumpers"
- note removed: "Row jumpers"
- moved on the sheet: JP_col1_B1, JP_col1_F1, JP_col2_B1, JP_col2_F1, JP_col3_B1, JP_col3_F1, JP_col4_B1, JP_col4_F1, JP_col5_B1, JP_col5_F1, JP_row1_B1, JP_row1_F1

Commit message: Finally cleaned up jumper situation
Parts:
- removed JP_col5_B1, JP_col5_F1: Jumper_2_Open, local-libraries:SolderJumper-2_P1.3mm_Open_RoundedPad1.0x1.5mm, symbol Jumper:Jumper_2_Open
- renumbered JP_row1_B1 to JP_col_B1, JP_row2_B1 to JP_col_B2, JP_row3_B1 to JP_col_B3, JP_row4_B1 to JP_col_B4, JP_row5_B1 to JP_col_B5, JP_row1_F1 to JP_col_F1, JP_row2_F1 to JP_col_F2, JP_row3_F1 to JP_col_F3, JP_row4_F1 to JP_col_F4, JP_row5_F1 to JP_col_F5, JP_col1_B1 to JP_row_B1, JP_col2_B1 to JP_row_B2, JP_col3_B1 to JP_row_B3, JP_col4_B1 to JP_row_B4, JP_col1_F1 to JP_row_F1, JP_col2_F1 to JP_row_F2, JP_col3_F1 to JP_row_F3, JP_col4_F1 to JP_row_F4
Connections:
- net col1_matrix: now also JP_col_B1.2 (B), JP_col_F1.1 (A); no longer JP_row_B1.1 (A), JP_row_F1.2 (B)
- net col2_matrix: now also JP_col_B2.2 (B), JP_col_F2.1 (A); no longer JP_row_B2.1 (A), JP_row_F2.2 (B)
- net col3_matrix: now also JP_col_B3.2 (B), JP_col_F3.1 (A); no longer JP_row_B3.1 (A), JP_row_F3.2 (B)
- net col4_matrix: now also JP_col_B4.2 (B), JP_col_F4.1 (A); no longer JP_row_B4.1 (A), JP_row_F4.2 (B)
- net col5_matrix: now also JP_col_B5.2 (B), JP_col_F5.1 (A)
- net row1_matrix: now also JP_row_B1.1 (A), JP_row_F1.2 (B); no longer JP_col_B1.2 (B), JP_col_F1.1 (A)
- net row2_matrix: now also JP_row_B2.1 (A), JP_row_F2.2 (B); no longer JP_col_B2.2 (B), JP_col_F2.1 (A)
- net row3_matrix: now also JP_row_B3.1 (A), JP_row_F3.2 (B); no longer JP_col_B3.2 (B), JP_col_F3.1 (A)
- net row4_matrix: now also JP_row_B4.1 (A), JP_row_F4.2 (B); no longer JP_col_B4.2 (B), JP_col_F4.1 (A)
- net row5_mcu_unused: now also U1.12 (P1.06)
- net batt renamed +5V
- no-connect marks 14 -> 13
Other:
- moved on the sheet: JP_col_B1, JP_col_B2, JP_col_B3, JP_col_B4, JP_col_B5, JP_col_F1, JP_col_F2, JP_col_F3, JP_col_F4, JP_col_F5, JP_row_B1, JP_row_B2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
